Commit message: Add GPS plugin

File: robot_boat_description_pkg/urdf/robot_boat.xacro (robot description, xacro)
@@ -6,5 +6,5 @@
 <xacro:property name="body_width" value="1.0"/>
 <xacro:property name="body_lenght" value="2.0"/>
-<xacro:property name="body_height" value="1.0"/>
+<xacro:property name="body_height" value="0.5"/>
 <xacro:property name="wheel_width" value="0.2"/>
 <xacro:property name="wheel_radius" value="0.1"/>
@@ -112,5 +112,5 @@
   </link>
   <joint name="front_yaw_joint" type="continuous">
-    <origin rpy="0 0 0" xyz="${body_lenght / 2 - 0.1} 0 -${body_height / 2 - 0.05 }" />
+    <origin rpy="0 0 0" xyz="${body_lenght / 2 - 0.1} 0 -${body_height / 2 - 0.02 }" />
     <parent link="chassis" />
     <child link="front_yaw_link" />
@@ -197,5 +197,5 @@
   </link>
   <joint name="back_yaw_joint" type="continuous">
-    <origin rpy="0 0 0" xyz="-${body_lenght / 2.0 - 0.1} 0 -${body_height / 2 - 0.05 }" />
+    <origin rpy="0 0 0" xyz="-${body_lenght / 2.0 - 0.1} 0 -${body_height / 2 - 0.02 }" />
     <parent link="chassis" />
     <child link="back_yaw_link" />
@@ -324,5 +324,5 @@
   </link>
   <joint name="laser_scan_link_joint" type="fixed">
-    <origin rpy="0 0 0" xyz="0.0 0.0 0.05"/>
+    <origin rpy="0 0 0" xyz="0.0 0.0 ${body_height/2}"/>
     <parent link="chassis"/>
     <child link="laser_scan_link"/>
@@ -358,5 +358,5 @@
         </ray>
         <always_on>true</always_on>
-        <visualize>false</visualize>
+        <visualize>true</visualize>
         <update_rate>10.0</update_rate>
         <plugin name="laser" filename="libgazebo_ros_ray_sensor.so">
@@ -369,3 +369,20 @@
     </sensor>
 </gazebo>
+  <!-- GPS plugin -->
+<gazebo reference="laser_scan_frame">
+    <sensor name="gps_sensor" type="gps">
+        <always_on>true</always_on>
+        <update_rate>1.0</update_rate>
+        <drift>2.0 2.0 2.0</drift>
+        <gaussiannoise>0.1 0.1 0.1</gaussiannoise>
+        <plugin name="gps_controller" filename="libgazebo_ros_gps_sensor.so">
+            <ros>
+                <namespace>/robot_boat</namespace>
+                <remapping>gps_controller/out:=gps</remapping>
+            </ros>
+            <frame_name>laser_scan_frame</frame_name>
+        </plugin>
+    </sensor>
+    <material>Gazebo/Grey</material>
+</gazebo>
 </robot>
