Commit message: Robot scaled to real size

File: robot_boat_description_pkg/urdf/robot_boat.gazebo.xacro (robot description, xacro)
@@ -3,29 +3,33 @@
     <xacro:macro name="gazebo_elements">
   <gazebo reference="left_wheel">
-    <kp>1000000000000000000000000000.0</kp>
-    <kd>1000000000000000000000000000.0</kd>
-    <mu1>10.0</mu1>
+    <kp>100000.0</kp>
+    <kd>100000.0</kd>
+    <mu1>15.0</mu1>
     <mu2>10.0</mu2>
+    <fdir1>1 1 1</fdir1>
     <material>Gazebo/Red</material>
   </gazebo>
   <gazebo reference="right_wheel">
-    <kp>1000000000000000000000000000.0</kp>
-    <kd>1000000000000000000000000000.0</kd>
-    <mu1>10.0</mu1>
+    <kp>100000.0</kp>
+    <kd>100000.0</kd>
+    <mu1>15.0</mu1>
     <mu2>10.0</mu2>
+    <fdir1>1 1 1</fdir1>
     <material>Gazebo/Green</material>
   </gazebo>
   <gazebo reference="front_pitch_link">
-    <kp>1000000000000000000000000000.0</kp>
-    <kd>1000000000000000000000000000.0</kd>
-    <mu1>1</mu1>
-    <mu2>0.5</mu2>
+    <kp>100000000000000000000.0</kp>
+    <kd>100000000000000000000.0</kd>
+    <mu1>5</mu1>
+    <mu2>5</mu2>
+    <fdir1>1 1 1</fdir1>
     <material>Gazebo/Purple</material>
   </gazebo>
   <gazebo reference="back_pitch_link">
-    <kp>1000000000000000000000000000.0</kp>
-    <kd>1000000000000000000000000000.0</kd>
-    <mu1>1</mu1>
-    <mu2>0.5</mu2>
+    <kp>100000000000000000000.0</kp>
+    <kd>100000000000000000000.0</kd>
+    <mu1>5</mu1>
+    <mu2>5</mu2>
+    <fdir1>1 1 1</fdir1>
     <material>Gazebo/Yellow</material>
   </gazebo>

File: robot_boat_description_pkg/urdf/robot_boat.xacro (robot description, xacro)
@@ -4,10 +4,11 @@
     <xacro:gazebo_elements />
 <!-- Properties -->
-<xacro:property name="body_width" value="0.1"/>
-<xacro:property name="body_lenght" value="0.1"/>
-<xacro:property name="body_height" value="0.1"/>
-<xacro:property name="wheel_width" value="0.001"/>
-<xacro:property name="wheel_radius" value="0.035"/>
-<xacro:property name="wheel_distance" value="0.035"/>
+<xacro:property name="body_width" value="1.0"/>
+<xacro:property name="body_lenght" value="2.0"/>
+<xacro:property name="body_height" value="1.0"/>
+<xacro:property name="wheel_width" value="0.2"/>
+<xacro:property name="wheel_radius" value="0.1"/>
+<xacro:property name="wheel_distance" value="body_width"/>
+<xacro:property name="caster_radius" value="0.1"/>
   <material name="red">
       <color rgba="1.0 0.0 0.0 1"/>
@@ -28,14 +29,14 @@
     <visual>
       <geometry>
-        <mesh filename="package://robot_boat_description_pkg/meshes/cute_cube.dae" scale="${body_width} ${body_lenght} ${body_height}"/>
+        <mesh filename="package://robot_boat_description_pkg/meshes/cute_cube.dae" scale="${body_lenght} ${body_width}  ${body_height}"/>
       </geometry>
     </visual>
     <collision>
       <geometry>
-        <box size="${body_width} ${body_lenght} ${body_height}"/>
+        <box size="${body_lenght} ${body_width} ${body_height}"/>
       </geometry>
     </collision>
     <inertial>
-      <mass value="0.5"/>
+      <mass value="0.1"/>
       <origin rpy="0 0 0" xyz="0 0 0"/>
       <inertia ixx="0.0008333333333333335" ixy="0" ixz="0" iyy="0.0008333333333333335" iyz="0" izz="0.0008333333333333335"/>
@@ -43,5 +44,5 @@
   </link>
   <joint name="base_link_joint" type="fixed">
-    <origin rpy="0 0 0" xyz="0 0 0" />
+    <origin rpy="0 0 0" xyz="0 0 ${body_height / 2.0}" />
     <parent link="base_link" />
     <child link="chassis" />
@@ -64,5 +65,5 @@
         <inertial>
             <origin rpy="0 1.5707 1.5707" xyz="0 0 0"/>
-            <mass value="0.05"/>
+            <mass value="0.1"/>
             <inertia ixx="1.531666666666667e-05" ixy="0" ixz="0" iyy="1.531666666666667e-05" iyz="0" izz="3.0625000000000006e-05"/>
         </inertial>
@@ -74,18 +75,18 @@
     <xacro:wheel wheel_name="right_wheel" />
   <joint name="joint_left_wheel" type="continuous">
-    <origin rpy="0 0 0" xyz="0 0.05 -0.025"/>
+    <origin rpy="0 0 0" xyz="0 ${body_width/2} -${body_height/2}"/>
     <child link="left_wheel"/>
     <parent link="chassis"/>
     <axis rpy="0 0 0" xyz="0 1 0"/>
     <limit effort="10000" velocity="1000"/>
-    <joint_properties damping="1.0" friction="1.0"/>
+    <joint_properties damping="10.0" friction="10.0"/>
   </joint>
   <joint name="joint_right_wheel" type="continuous">
-    <origin rpy="0 0 0" xyz="0 -0.05 -0.025"/>
+    <origin rpy="0 0 0" xyz="0 -${body_width/2} -${body_height/2}"/>
     <child link="right_wheel"/>
     <parent link="chassis"/>
     <axis rpy="0 0 0" xyz="0 1 0"/>
     <limit effort="10000" velocity="1000"/>
-    <joint_properties damping="1.0" friction="1.0"/>
+    <joint_properties damping="10.0" friction="10.0"/>
   </joint>
   <!-- Caster Wheel Front -->
@@ -111,5 +112,5 @@
   </link>
   <joint name="front_yaw_joint" type="continuous">
-    <origin rpy="0 0 0" xyz="0.04 0 -0.05" />
+    <origin rpy="0 0 0" xyz="${body_lenght / 2 - 0.1} 0 -${body_height / 2 - 0.05 }" />
     <parent link="chassis" />
     <child link="front_yaw_link" />
@@ -150,5 +151,5 @@
       <origin rpy="0 1.5707 1.5707" xyz="0 0 0"/>
       <geometry>
-        <sphere radius="0.010"/>
+        <sphere radius="${caster_radius}"/>
       </geometry>
       <material name="green_dark"/>
@@ -157,5 +158,5 @@
       <origin rpy="0 1.5707 1.5707" xyz="0 0 0"/>
       <geometry>
-        <sphere radius="0.010"/>
+        <sphere radius="${caster_radius}"/>
       </geometry>
     </collision>
@@ -196,5 +197,5 @@
   </link>
   <joint name="back_yaw_joint" type="continuous">
-    <origin rpy="0 0 0" xyz="-0.04 0 -0.05" />
+    <origin rpy="0 0 0" xyz="-${body_lenght / 2.0 - 0.1} 0 -${body_height / 2 - 0.05 }" />
     <parent link="chassis" />
     <child link="back_yaw_link" />
@@ -235,5 +236,5 @@
       <origin rpy="0 1.5707 1.5707" xyz="0 0 0"/>
       <geometry>
-        <sphere radius="0.010"/>
+        <sphere radius="${caster_radius}"/>
       </geometry>
       <material name="green_light"/>
@@ -242,5 +243,5 @@
       <origin rpy="0 1.5707 1.5707" xyz="0 0 0"/>
       <geometry>
-        <sphere radius="0.010"/>
+        <sphere radius="${caster_radius}"/>
       </geometry>
     </collision>

Commit message: Corrected robot dynamics

File: robot_boat_description_pkg/urdf/robot_boat.gazebo.xacro (robot description, xacro)
@@ -3,33 +3,23 @@
     <xacro:macro name="gazebo_elements">
   <gazebo reference="left_wheel">
-    <kp>100000.0</kp>
-    <kd>100000.0</kd>
-    <mu1>15.0</mu1>
-    <mu2>10.0</mu2>
-    <fdir1>1 1 1</fdir1>
+    <self_collide>1</self_collide>
+    <mu1>0.3</mu1>
+    <mu2>0.1</mu2>
     <material>Gazebo/Red</material>
   </gazebo>
   <gazebo reference="right_wheel">
-    <kp>100000.0</kp>
-    <kd>100000.0</kd>
-    <mu1>15.0</mu1>
-    <mu2>10.0</mu2>
-    <fdir1>1 1 1</fdir1>
+    <self_collide>1</self_collide>
+    <mu1>0.3</mu1>
+    <mu2>0.1</mu2>
     <material>Gazebo/Green</material>
   </gazebo>
   <gazebo reference="front_pitch_link">
-    <kp>100000000000000000000.0</kp>
-    <kd>100000000000000000000.0</kd>
-    <mu1>5</mu1>
-    <mu2>5</mu2>
-    <fdir1>1 1 1</fdir1>
+    <mu1>0.05</mu1>
+    <mu2>0.05</mu2>
     <material>Gazebo/Purple</material>
   </gazebo>
   <gazebo reference="back_pitch_link">
-    <kp>100000000000000000000.0</kp>
-    <kd>100000000000000000000.0</kd>
-    <mu1>5</mu1>
-    <mu2>5</mu2>
-    <fdir1>1 1 1</fdir1>
+    <mu1>0.05</mu1>
+    <mu2>0.05</mu2>
     <material>Gazebo/Yellow</material>
   </gazebo>

File: robot_boat_description_pkg/urdf/robot_boat.xacro (robot description, xacro)
@@ -9,5 +9,5 @@
 <xacro:property name="wheel_width" value="0.2"/>
 <xacro:property name="wheel_radius" value="0.1"/>
-<xacro:property name="wheel_distance" value="body_width"/>
+<xacro:property name="wheel_distance" value="${body_width}"/>
 <xacro:property name="caster_radius" value="0.1"/>
   <material name="red">
@@ -38,7 +38,7 @@
     </collision>
     <inertial>
-      <mass value="0.1"/>
+      <mass value="30"/>
       <origin rpy="0 0 0" xyz="0 0 0"/>
-      <inertia ixx="0.0008333333333333335" ixy="0" ixz="0" iyy="0.0008333333333333335" iyz="0" izz="0.0008333333333333335"/>
+      <inertia ixx="3.125" ixy="0" ixz="0" iyy="10.62" iyz="0" izz="12.5"/>
     </inertial>
   </link>
@@ -65,6 +65,6 @@
         <inertial>
             <origin rpy="0 1.5707 1.5707" xyz="0 0 0"/>
-            <mass value="0.1"/>
-            <inertia ixx="1.531666666666667e-05" ixy="0" ixz="0" iyy="1.531666666666667e-05" iyz="0" izz="3.0625000000000006e-05"/>
+            <mass value="1"/>
+            <inertia ixx="0.0058" ixy="0" ixz="0" iyy="0.0058" iyz="0" izz="0.005"/>
         </inertial>
     </link>
@@ -79,6 +79,6 @@
     <parent link="chassis"/>
     <axis rpy="0 0 0" xyz="0 1 0"/>
-    <limit effort="10000" velocity="1000"/>
-    <joint_properties damping="10.0" friction="10.0"/>
+    <limit effort="1000" velocity="1000"/>
+    <joint_properties damping="0" friction="0.1"/>
   </joint>
   <joint name="joint_right_wheel" type="continuous">
@@ -87,6 +87,6 @@
     <parent link="chassis"/>
     <axis rpy="0 0 0" xyz="0 1 0"/>
-    <limit effort="10000" velocity="1000"/>
-    <joint_properties damping="10.0" friction="10.0"/>
+    <limit effort="1000" velocity="1000"/>
+    <joint_properties damping="0" friction="0.1"/>
   </joint>
   <!-- Caster Wheel Front -->
@@ -265,5 +265,5 @@
     <plugin name="box_bot_joint_state" filename="libgazebo_ros_joint_state_publisher.so">
       <ros>
-          <remapping>~/out:=joint_states</remapping>
+          <remapping>~/out:=robot_boat/joint_states</remapping>
       </ros>
       <update_rate>30</update_rate>
@@ -285,11 +285,11 @@
             <remapping>/odom:=odom</remapping>
         </ros>
-        <update_rate>50</update_rate>
+        <update_rate>10</update_rate>
         <!-- Wheel joints -->
         <left_joint>joint_left_wheel</left_joint>
         <right_joint>joint_right_wheel</right_joint>
         <!-- Kinematics -->
-        <wheel_separation>0.1</wheel_separation>
-        <wheel_diameter>0.07</wheel_diameter>
+        <wheel_separation>${wheel_distance}</wheel_separation>
+        <wheel_diameter>${wheel_radius*2}</wheel_diameter>
         <publish_odom>true</publish_odom>
         <!-- TF frames -->
@@ -299,10 +299,22 @@
         <robot_base_frame>base_link</robot_base_frame>
         <!-- Limits -->
-        <max_wheel_torque>1.0</max_wheel_torque>
-        <max_wheel_acceleration>2.0</max_wheel_acceleration>
+        <max_wheel_torque>100.0</max_wheel_torque>
+        <max_wheel_acceleration>0.2</max_wheel_acceleration>
     </plugin>
   </gazebo>
     <!-- Laser Position Control-->
   <link name="laser_scan_link">
+    <inertial>
+      <mass value="0.01"/>
+      <origin rpy="0 0 0" xyz="0 0 0.0204"/>
+      <inertia ixx="6.066578520833334e-06" ixy="0" ixz="0" iyy="6.072950163333333e-06" iyz="0" izz="9.365128684166666e-06"/>
+    </inertial>
+  </link>
+  <joint name="laser_scan_link_joint" type="fixed">
+    <origin rpy="0 0 0" xyz="0.0 0.0 ${body_height/2}"/>
+    <parent link="chassis"/>
+    <child link="laser_scan_link"/>
+  </joint>
+  <link name="laser_scan_frame">
     <visual>
       <origin rpy="0 0 0" xyz="0 0 0"/>
@@ -323,20 +335,15 @@
     </inertial>
   </link>
-  <joint name="laser_scan_link_joint" type="fixed">
-    <origin rpy="0 0 0" xyz="0.0 0.0 ${body_height/2}"/>
-    <parent link="chassis"/>
-    <child link="laser_scan_link"/>
-    <axis xyz="0 0 1"/>
-    <limit lower="-0.1" upper="0.0" effort="20.0" velocity="2.0"/>
-    <dynamics damping="0.1" friction="1.0"/>
-  </joint>
-  <link name="laser_scan_frame">
-  </link>
   <joint name="laser_scan_frame_joint" type="fixed">
-    <origin rpy="0 0 0" xyz="0 0 0.03"/>
+    <origin rpy="0 0 0" xyz="0 0 0.2"/>
     <parent link="laser_scan_link"/>
     <child link="laser_scan_frame"/>
     <axis xyz="0 0 0"/>
   </joint>
+    <!--
+  <gazebo reference="laser_scan_frame_joint">
+    <preserveFixedJoint>true</preserveFixedJoint>
+  </gazebo>
+  -->
   <!-- Lser plugin -->
 <gazebo reference="laser_scan_frame">
@@ -353,5 +360,5 @@
           </scan>
           <range>
-            <min>0.2</min>
+            <min>1.2</min>
             <max>20</max>
           </range>
@@ -359,5 +366,5 @@
         <always_on>true</always_on>
         <visualize>false</visualize>
-        <update_rate>10.0</update_rate>
+        <update_rate>5</update_rate>
         <plugin name="laser" filename="libgazebo_ros_ray_sensor.so">
           <ros>
@@ -366,4 +373,5 @@
           </ros>
           <output_type>sensor_msgs/LaserScan</output_type>
+          <frame_name>laser_scan_frame</frame_name>
         </plugin>
     </sensor>
